File: pp/power_switches/power_switches.kicad_pcb (KiCad board)
At the start: 2 copper layers, 8 parts, among them J1 Screw_Terminal_1x02, J2 Screw_Terminal_1x02, P1 CONN_01X02, U1 MOC3063M

Commit message: силовые ключи
Parts:
- J1, J2: footprint Connectors:bornier2 -> Connectors_Terminal_Blocks:TerminalBlock_Pheonix_MPT-2.54mm_2pol
- P1: footprint Connectors_Terminal_Blocks:TerminalBlock_Pheonix_MPT-2.54mm_2pol -> Socket_Strips:Socket_Strip_Straight_1x02_Pitch2.54mm
- R1: value 1k -> 100; footprint Resistors_THT:R_Axial_DIN0309_L9.0mm_D3.2mm_P15.24mm_Horizontal -> Resistors_SMD:R_1206
- R2: footprint Resistors_THT:R_Axial_DIN0309_L9.0mm_D3.2mm_P15.24mm_Horizontal -> Resistors_SMD:R_1206
- moved J1 74.1 mm to (109.0, 51.0)
- moved J2 74.0 mm to (109.0, 64.0)
- moved R2 71.6 mm to (82.3, 44.5)
- moved D1 63.6 mm to (92.0, 58.0)
- moved R1 57.7 mm to (65.5, 46.0)
- moved U1 50.5 mm to (73.0, 55.0)
- moved P1 39.1 mm to (58.8, 53.6), turned to 180 degrees
- moved C1 29.1 mm to (68.0, 63.0)
Routing:
- net Net-(D1-Pad1): track 0.00 -> 20.8 mm
- net Net-(D1-Pad2): track 0.00 -> 19.7 mm
- net Net-(D1-Pad3): track 0.00 -> 11.6 mm
- net Net-(C1-Pad2): track 0.00 -> 11.0 mm
- net Net-(J1-Pad1): track 0.00 -> 10.5 mm
Other:
- board outline added: 60 x 30 mm
- net class 220-10A added: clearance 0.3, trace_width 1.1, via_dia 0.6, via_drill 0.4
